Commit message: Version 1.0

File: donatello_description/urdf/extensions.urdf.xacro (robot description, xacro)
@@ -71,5 +71,5 @@
         <origin xyz="0.003 -0.009 0.083" rpy="0 ${pi/2} ${pi/4}" />
         <geometry>
-          <mesh filename="package://robomaster_description/meshes/intelligent_controller.dae" />
+          <mesh filename="file:$(find robomaster_description)/meshes/intelligent_controller.dae" />
         </geometry>
       </visual>

File: donatello_description/urdf/sensors.urdf.xacro (robot description, xacro)
@@ -3,10 +3,10 @@
   <xacro:macro name="add_gazebo_sensors" params="tf_prefix=''">
     <xacro:sensor_d435i_gazebo_sim light_mode="true" />
-    <xacro:sensor_rplidar_a2_m12_gazebo_sim prefix="rear" />
+    <xacro:sensor_rplidar_a2_m12_gazebo_sim prefix="rear" range_min="0.25" />
     <plugin name="donatello_joint_state" filename="libgazebo_ros_joint_state_publisher.so">
       <ros>
         <remapping>~/out:=joint_states</remapping>
       </ros>
-      <update_rate>25</update_rate>
+      <update_rate>50</update_rate>
       <joint_name>donatello_front_left_wheel_joint</joint_name>
       <joint_name>donatello_front_right_wheel_joint</joint_name>
@@ -21,7 +21,4 @@
         <back_left_joint>donatello_rear_left_wheel_joint</back_left_joint>
         <back_right_joint>donatello_rear_right_wheel_joint</back_right_joint>
-        <wheel_separation>0.2</wheel_separation>
-        <wheelbase>0.2</wheelbase>
-        <wheel_radius>0.5</wheel_radius>
         <min_acceleration>-5</min_acceleration>
         <max_acceleration>5</max_acceleration>
@@ -32,4 +29,18 @@
         <child_frame_id>base_link</child_frame_id>
         <odom_publish_frequency>50</odom_publish_frequency>
+        <!-- play with these three to simulate bad dometry -->
+        <wheel_separation>0.20</wheel_separation>
+        <wheelbase>0.20</wheelbase>
+        <wheel_radius>0.050</wheel_radius>
+      </plugin>
+    </gazebo>
+    <gazebo>
+      <plugin filename="gz-sim-joint-state-publisher-system"
+        name="gz::sim::systems::JointStatePublisher">
+        <topic>joint_states</topic>
+          <joint_name>donatello_front_left_wheel_joint</joint_name>
+          <joint_name>donatello_front_right_wheel_joint</joint_name>
+          <joint_name>donatello_rear_left_wheel_joint</joint_name>
+          <joint_name>donatello_rear_right_wheel_joint</joint_name>
       </plugin>
     </gazebo>
