Commit message: tf change

File: donatello_description/urdf/donatello.urdf.xacro (robot description, xacro)
@@ -8,11 +8,5 @@
   <!-- setting a prefix to avoid a name conflict between the robot description and
   the realsense sensor description. -->
-  <xacro:property name="tf_prefix" value="donatello_" />
-  <!-- creating a base link frame to use standard naming despite the prefix -->
-  <link name="base_link" />
-  <joint name="base_link_joint" type="fixed">
-    <parent link="base_link" />
-    <child link="donatello_base_link" />
-  </joint>
+  <xacro:property name="tf_prefix" value="donatello/" />
   <xacro:include filename="common_colors.urdf.xacro" />
   <xacro:include filename="$(find robomaster_description)/urdf/base.urdf.xacro" />

File: donatello_description/urdf/sensors.urdf.xacro (robot description, xacro)
@@ -9,16 +9,16 @@
       </ros>
       <update_rate>50</update_rate>
-      <joint_name>donatello_front_left_wheel_joint</joint_name>
-      <joint_name>donatello_front_right_wheel_joint</joint_name>
-      <joint_name>donatello_rear_left_wheel_joint</joint_name>
-      <joint_name>donatello_rear_right_wheel_joint</joint_name>
+      <joint_name>donatello/front_left_wheel_joint</joint_name>
+      <joint_name>donatello/front_right_wheel_joint</joint_name>
+      <joint_name>donatello/rear_left_wheel_joint</joint_name>
+      <joint_name>donatello/rear_right_wheel_joint</joint_name>
     </plugin>
     <gazebo>
       <plugin name="ignition::gazebo::systems::MecanumDrive"
         filename="ignition-gazebo-mecanum-drive-system">
-        <front_left_joint>donatello_front_left_wheel_joint</front_left_joint>
-        <front_right_joint>donatello_front_right_wheel_joint</front_right_joint>
-        <back_left_joint>donatello_rear_left_wheel_joint</back_left_joint>
-        <back_right_joint>donatello_rear_right_wheel_joint</back_right_joint>
+        <front_left_joint>donatello/front_left_wheel_joint</front_left_joint>
+        <front_right_joint>donatello/front_right_wheel_joint</front_right_joint>
+        <back_left_joint>donatello/rear_left_wheel_joint</back_left_joint>
+        <back_right_joint>donatello/rear_right_wheel_joint</back_right_joint>
         <min_acceleration>-5</min_acceleration>
         <max_acceleration>5</max_acceleration>
@@ -26,6 +26,6 @@
         <odom_topic>odom</odom_topic>
         <tf_topic>tf</tf_topic>
-        <frame_id>odom</frame_id>
-        <child_frame_id>base_link</child_frame_id>
+        <frame_id>donatello/odom</frame_id>
+        <child_frame_id>donatello/base_link</child_frame_id>
         <odom_publish_frequency>50</odom_publish_frequency>
         <!-- play with these three to simulate bad dometry -->
@@ -40,5 +40,5 @@
         filename="ignition-gazebo-odometry-publisher-system">
         <odom_frame>map</odom_frame>
-        <robot_base_frame>base_link</robot_base_frame>
+        <robot_base_frame>donatello/base_link</robot_base_frame>
         <odom_publish_frequency>20</odom_publish_frequency>
         <odom_topic>ground_truth</odom_topic>
@@ -50,8 +50,8 @@
         name="gz::sim::systems::JointStatePublisher">
         <topic>joint_states</topic>
-          <joint_name>donatello_front_left_wheel_joint</joint_name>
-          <joint_name>donatello_front_right_wheel_joint</joint_name>
-          <joint_name>donatello_rear_left_wheel_joint</joint_name>
-          <joint_name>donatello_rear_right_wheel_joint</joint_name>
+          <joint_name>donatello/front_left_wheel_joint</joint_name>
+          <joint_name>donatello/front_right_wheel_joint</joint_name>
+          <joint_name>donatello/rear_left_wheel_joint</joint_name>
+          <joint_name>donatello/rear_right_wheel_joint</joint_name>
       </plugin>
     </gazebo>

Commit message: Update drivers for new hardware

File: donatello_description/urdf/donatello.urdf.xacro (robot description, xacro)
@@ -2,6 +2,4 @@
 <robot xmlns:xacro="http://www.ros.org/wiki/xacro" name="donatello">
   <xacro:arg name="camera_yaw" default="0.0" />
-  <xacro:arg name="dummy_arm" default="true" />
-  <xacro:property name="dummy_arm_param" value="$(arg dummy_arm)" />
   <xacro:property name="package_name" value="donatello_description" />
   <xacro:property name="robot_name" value="donatello" />
@@ -15,29 +13,13 @@
   <xacro:include filename="$(find robomaster_description)/urdf/extension.urdf.xacro" />
   <xacro:include filename="$(find robomaster_description)/urdf/tof.urdf.xacro" />
-  <!-- use the alternate dummy arm with static articulations -->
-  <xacro:if value="${dummy_arm_param == True}">
-    <xacro:include
-      filename="$(find robomaster_description)/urdf/alternate/arm.urdf.xacro" />
-    <xacro:include
-      filename="$(find robomaster_description)/urdf/alternate/gripper.urdf.xacro" />
-  </xacro:if>
-  <!-- use the original articulated arm -->
-  <xacro:unless value="${dummy_arm_param == True}">
-    <xacro:include
-      filename="$(find robomaster_description)/urdf/arm.urdf.xacro" />
-    <xacro:include
-      filename="$(find robomaster_description)/urdf/gripper.urdf.xacro" />
-  </xacro:unless>
   <xacro:include filename="extensions.urdf.xacro" />
   <xacro:include filename="sensors.urdf.xacro" />
-  <xacro:include filename="$(find yolo_realsense2_models)/urdf/sensor_d435i.urdf.xacro" />
-  <xacro:include filename="$(find yolo_realsense2_models)/urdf/sensor_d435i_gazebo_sim.urdf.xacro" />
+  <xacro:include filename="$(find yolo_realsense2_models)/urdf/sensor_d455.urdf.xacro" />
+  <xacro:include filename="$(find yolo_realsense2_models)/urdf/sensor_d455_gazebo_sim.urdf.xacro" />
   <xacro:include filename="$(find yolo_rplidar_models)/urdf/sensor_rplidar_a2_m12.urdf.xacro" />
   <xacro:include
     filename="$(find yolo_rplidar_models)/urdf/sensor_rplidar_a2_m12_gazebo_sim.urdf.xacro" />
   <xacro:base tf_prefix="${tf_prefix}" />
-  <xacro:arm tf_prefix="${tf_prefix}" />
-  <xacro:camera tf_prefix="${tf_prefix}" mount="arm" camera_yaw="$(arg camera_yaw)" />
-  <xacro:gripper tf_prefix="${tf_prefix}" />
+  <!-- <xacro:camera tf_prefix="${tf_prefix}" mount="arm" camera_yaw="$(arg camera_yaw)" /> -->
   <xacro:extension tf_prefix="${tf_prefix}" use_rear_extension="false" />
   <xacro:add_tof index="0" tf_prefix="${tf_prefix}" />
@@ -47,5 +29,5 @@
   <xacro:lidar tf_prefix="${tf_prefix}" />
   <xacro:depth_camera tf_prefix="${tf_prefix}" />
-  <xacro:controller tf_prefix="${tf_prefix}" />
+  <!-- <xacro:controller tf_prefix="${tf_prefix}" /> -->
   <xacro:add_gazebo_sensors tf_prefix="${tf_prefix}" />
 </robot>

File: donatello_description/urdf/extensions.urdf.xacro (robot description, xacro)
@@ -2,23 +2,7 @@
 <robot xmlns:xacro="http://playerstage.sourceforge.net/gazebo/xmlschema/#xacro">
   <xacro:macro name="lidar" params="tf_prefix=''">
-    <joint name="${tf_prefix}arm_base_to_deck_joint" type="fixed">
-      <origin xyz="-0.115 0.00 0.0070" rpy="0 0 -${pi/2}" />
-      <parent link="${tf_prefix}arm_base_link" />
-      <child link="${tf_prefix}cpu_lidar_shelves" />
-    </joint>
-    <link name="${tf_prefix}cpu_lidar_shelves">
-      <inertial>
-        <mass value="0.01" />
-        <inertia ixx="0.01" ixy="0" ixz="0" iyy="0.01" iyz="0" izz="0.01" />
-      </inertial>
-      <visual>
-        <geometry>
-          <mesh filename="file:$(find donatello_description)/meshes/lidar_cpu_shelves.dae" />
-        </geometry>
-      </visual>
-    </link>
     <joint name="${tf_prefix}lidar_base_link_joint" type="fixed">
-      <origin xyz="0 0 0.003" rpy="0 0 0" />
-      <parent link="${tf_prefix}cpu_lidar_shelves" />
+      <origin xyz="0.005 0 0.0" rpy="0 0 0" />
+      <parent link="${tf_prefix}extension_base_link" />
       <child link="${tf_prefix}lidar_base_link" />
     </joint>
@@ -28,26 +12,27 @@
   <xacro:macro name="depth_camera" params="tf_prefix=''">
     <joint name="${tf_prefix}camera_support_joint" type="fixed">
-      <origin xyz="0.018 0.0 -0.01" rpy="0 0 0" />
-      <parent link="${tf_prefix}gripper_link_link" />
-      <child link="${tf_prefix}camera_support_link" />
+      <origin xyz="0.005 0.0 0.047" rpy="0 0 0" />
+      <parent link="${tf_prefix}extension_base_link" />
+      <child link="${tf_prefix}upper_deck_link" />
     </joint>
-    <link name="${tf_prefix}camera_support_link">
+    <link name="${tf_prefix}upper_deck_link">
       <inertial>
         <mass value="0.01" />
         <inertia ixx="0.01" ixy="0" ixz="0" iyy="0.01" iyz="0" izz="0.01" />
       </inertial>
-      <visual>
+      <!-- <visual>
         <geometry>
-          <mesh filename="file:$(find donatello_description)/meshes/depth_camera_support.dae" />
+          <mesh filename="file:$(find donatello_description)/meshes/donatello_upper_deck.dae" />
         </geometry>
-      </visual>
+        <origin xyz="0.0 0.0 0.0" rpy="3.14159265359 0 0" />
+      </visual> -->
     </link>
     <joint name="${tf_prefix}camera_mount_joint" type="fixed">
-      <origin xyz="0.0372 0 0.001" rpy="0 0 0" />
-      <parent link="${tf_prefix}camera_support_link" />
+      <origin xyz="-0.073 0 0.184" rpy="0 0 0" />
+      <parent link="${tf_prefix}upper_deck_link" />
       <child link="${tf_prefix}depth_camera_mount_link" />
     </joint>
     <link name="${tf_prefix}depth_camera_mount_link" />
-    <xacro:sensor_d435i parent="${tf_prefix}depth_camera_mount_link" use_nominal_extrinsics="true" />
+    <xacro:sensor_d455 parent="${tf_prefix}depth_camera_mount_link" use_nominal_extrinsics="true" />
   </xacro:macro>
   <xacro:macro name="controller" params="tf_prefix=''">

File: donatello_description/urdf/sensors.urdf.xacro (robot description, xacro)
@@ -2,5 +2,5 @@
 <robot xmlns:xacro="http://playerstage.sourceforge.net/gazebo/xmlschema/#xacro">
   <xacro:macro name="add_gazebo_sensors" params="tf_prefix=''">
-    <xacro:sensor_d435i_gazebo_sim light_mode="true" />
+    <xacro:sensor_d455_gazebo_sim light_mode="true" />
     <xacro:sensor_rplidar_a2_m12_gazebo_sim prefix="rear" range_min="0.25" />
     <plugin name="donatello_joint_state" filename="libgazebo_ros_joint_state_publisher.so">
